Commit message: close gripper

File: robots/ur5/urdf/ur5_pen.urdf (robot description, URDF)
Before this commit: robot ur5_robot, 24 links, 23 joints
Joints:
- joint finger_joint: origin xyz=0 -0.0306011 0.054904 rpy=0 0 3.14159265359 -> xyz=0 -0.0306011 0.054904 rpy=0.67 0 3.14159265359
- joint left_inner_finger_joint: origin xyz=0 0.0061 0.0471 rpy=0 0 0 -> xyz=0 0.0061 0.0471 rpy=-0.67 0 0
- joint left_inner_knuckle_joint: origin xyz=0 -0.0127 0.06142 rpy=0 0 3.14159265359 -> xyz=0 -0.0127 0.06142 rpy=0.67 0 3.14159265359
- joint right_inner_finger_joint: origin xyz=0 0.0061 0.0471 rpy=0 0 0 -> xyz=0 0.0061 0.0471 rpy=-0.67 0 0
- joint right_inner_knuckle_joint: origin xyz=0 0.0127 0.06142 rpy=0 0 0.0 -> xyz=0 0.0127 0.06142 rpy=0.67 0 0.0
- joint right_outer_knuckle_joint: origin xyz=0 0.0306011 0.054904 rpy=0 0 0 -> xyz=0 0.0306011 0.054904 rpy=0.67 0 0
